File: hardware/pmod-breakout/pmod-breakout.sch (KiCad schematic (older format))
At the start: 7 parts, among them J1 Feather, J2 PMOD, J3 PMOD

Commit message: updated board + pmod
Parts:
- removed D?: LED_RGBA, symbol josh-symbols:LED_RGBA
- removed R?: 10K, symbol Device:R
- removed RN?: 330R, symbol Device:R_Pack04
- removed SW?: SW_Push, symbol Switch:SW_Push
Connections:
- net USR_BTN: no longer names the net of J1.25 (IO19)
- net nLED_BLUE: no longer names the net of J1.13 (IO8|MISO)
- net nLED_GREEN: no longer names the net of J1.14 (IO9|RX)
- net nLED_RED: no longer names the net of J1.15 (IO10|TX)
- no-connect marks 7 -> 9
Other:
- note removed: "Bonus!"
Changed lines of the file:
@@
 EESchema Schematic File Version 4
+LIBS:pmod-breakout-cache
 EELAYER 29 0
 EELAYER END
@@
 Text Notes 4050 1050 0    197  ~ 0
 Feather to Dual PMOD
-$Comp
-L josh-symbols:LED_RGBA D?
-U 1 1 5D182266
-P 8550 2625
-F 0 "D?" H 8550 3122 50  0000 C CNN
-F 1 "LED_RGBA" H 8550 3031 50  0000 C CNN
-F 2 "" H 8550 2575 50  0001 C CNN
-F 3 "~" H 8550 2575 50  0001 C CNN
-	1    8550 2625
-	1    0    0    -1
-$EndComp
-Wire Wire Line
-	8750 2625 8875 2625
-Wire Wire Line
-	8875 2625 8875 2475
-$Comp
-L power:+3V3 #PWR?
-U 1 1 5D185049
-P 8875 2475
-F 0 "#PWR?" H 8875 2325 50  0001 C CNN
-F 1 "+3V3" H 8890 2648 50  0000 C CNN
-F 2 "" H 8875 2475 50  0001 C CNN
-F 3 "" H 8875 2475 50  0001 C CNN
-	1    8875 2475
-	1    0    0    -1
-$EndComp
-$Comp
-L Device:R_Pack04 RN?
-U 1 1 5D187D48
-P 8000 2675
-F 0 "RN?" V 7583 2675 50  0000 C CNN
-F 1 "330R" V 7674 2675 50  0000 C CNN
-F 2 "" V 8275 2675 50  0001 C CNN
-F 3 "~" H 8000 2675 50  0001 C CNN
-	1    8000 2675
-	0    1    1    0
-$EndComp
-Wire Wire Line
-	8200 2475 8275 2475
-Wire Wire Line
-	8275 2475 8275 2425
-Wire Wire Line
-	8275 2425 8350 2425
-Wire Wire Line
-	8200 2575 8275 2575
-Wire Wire Line
-	8275 2575 8275 2625
-Wire Wire Line
-	8275 2625 8350 2625
-Wire Wire Line
-	8200 2775 8275 2775
-Wire Wire Line
-	8275 2775 8275 2825
-Wire Wire Line
-	8275 2825 8350 2825
-NoConn ~ 8200 2675
-NoConn ~ 7800 2675
-Text Label 7325 2475 0    50   ~ 0
-nLED_RED
-Wire Wire Line
-	7325 2475 7800 2475
-Text Label 7325 2575 0    50   ~ 0
-nLED_GREEN
-Wire Wire Line
-	7325 2575 7800 2575
-Text Label 7325 2775 0    50   ~ 0
-nLED_BLUE
-Wire Wire Line
-	7325 2775 7800 2775
-Text Notes 7950 1900 0    118  ~ 0
-Bonus!
-$Comp
-L Switch:SW_Push SW?
-U 1 1 5D1AB359
-P 8275 3450
-F 0 "SW?" H 8275 3735 50  0000 C CNN
-F 1 "SW_Push" H 8275 3644 50  0000 C CNN
-F 2 "" H 8275 3650 50  0001 C CNN
-F 3 "~" H 8275 3650 50  0001 C CNN
-	1    8275 3450
-	1    0    0    -1
-$EndComp
-Text Label 7450 3450 0    50   ~ 0
-USR_BTN
-Wire Wire Line
-	7450 3450 7925 3450
-Wire Wire Line
-	8475 3450 8875 3450
-Wire Wire Line
-	8875 3450 8875 3225
-$Comp
-L power:+3V3 #PWR?
-U 1 1 5D1B606D
-P 8875 3225
-F 0 "#PWR?" H 8875 3075 50  0001 C CNN
-F 1 "+3V3" H 8890 3398 50  0000 C CNN
-F 2 "" H 8875 3225 50  0001 C CNN
-F 3 "" H 8875 3225 50  0001 C CNN
-	1    8875 3225
-	1    0    0    -1
-$EndComp
-$Comp
-L Device:R R?
-U 1 1 5D1B8D95
-P 7925 3675
-F 0 "R?" H 7995 3721 50  0000 L CNN
-F 1 "10K" H 7995 3630 50  0000 L CNN
-F 2 "" V 7855 3675 50  0001 C CNN
-F 3 "~" H 7925 3675 50  0001 C CNN
-	1    7925 3675
-	1    0    0    -1
-$EndComp
-Wire Wire Line
-	7925 3525 7925 3450
-Connection ~ 7925 3450
-Wire Wire Line
-	7925 3450 8075 3450
-$Comp
-L power:GND #PWR?
-U 1 1 5D1BB728
-P 7925 3850
-F 0 "#PWR?" H 7925 3600 50  0001 C CNN
-F 1 "GND" H 7930 3677 50  0000 C CNN
-F 2 "" H 7925 3850 50  0001 C CNN
-F 3 "" H 7925 3850 50  0001 C CNN
-	1    7925 3850
-	1    0    0    -1
-$EndComp
-Wire Wire Line
-	7925 3850 7925 3825
-Text Label 3350 2875 0    50   ~ 0
-USR_BTN
-Wire Wire Line
-	3350 2875 3775 2875
-Text Label 5300 2175 2    50   ~ 0
-nLED_RED
-Wire Wire Line
-	5300 2175 4825 2175
-Text Label 5300 2275 2    50   ~ 0
-nLED_GREEN
-Wire Wire Line
-	5300 2275 4825 2275
-Text Label 5300 2375 2    50   ~ 0
-nLED_BLUE
-Wire Wire Line
-	5300 2375 4825 2375
+NoConn ~ 4825 2175
+NoConn ~ 4825 2275
+NoConn ~ 4825 2375
+NoConn ~ 3775 2875
 $EndSCHEMATC

Commit message: changes to make everything work with new library setup
Parts:
- removed J1: Feather, josh-footprints:PCB_FeatherWing, symbol josh-symbols:Feather
- added J1: Feather, josh-connectors:featherwing, symbol josh-mechnanical:Feather
- J2, J3: footprint josh-footprints:PMOD_HOST -> josh-connectors:PMOD_HOST
Connections:
- net +3V3: now also J1.2 (3V3)
- net GND: now also J1.16 (NC), J1.4 (GND)
- net P1_1: now also J1.12 (IO7|MOSI)
- net P1_10: now also J1.5 (IO0)
- net P1_2: now also J1.10 (IO5)
- net P1_3: now also J1.8 (IO3)
- net P1_4: now also J1.6 (IO1)
- net P1_7: now also J1.11 (IO6|SCK)
- net P1_8: now also J1.9 (IO4)
- net P1_9: now also J1.7 (IO2)
- net P2_1: now also J1.17 (IO11|SDA)
- net P2_10: now also J1.24 (IO18)
- net P2_2: now also J1.19 (IO13)
- net P2_3: now also J1.21 (IO15)
- net P2_4: now also J1.23 (IO17)
- net P2_7: now also J1.18 (IO12|SCL)
- net P2_8: now also J1.20 (IO14)
- net P2_9: now also J1.22 (IO16)
Changed lines of the file:
@@
 $EndDescr
-$Comp
-L josh-symbols:Feather J1
-U 1 1 5D133E2D
-P 4275 2775
-F 0 "J1" H 4300 3740 50  0000 C CNN
-F 1 "Feather" H 4300 3649 50  0000 C CNN
-F 2 "josh-footprints:PCB_FeatherWing" H 4475 1825 50  0001 C CNN
-F 3 "" H 4475 1825 50  0001 C CNN
-	1    4275 2775
-	1    0    0    -1
-$EndComp
 $Comp
 L Connector_Generic:Conn_02x06_Top_Bottom J2
@@
 F 0 "J2" H 6350 2717 50  0000 C CNN
 F 1 "PMOD" H 6350 2626 50  0000 C CNN
-F 2 "josh-footprints:PMOD_HOST" H 6300 2300 50  0001 C CNN
+F 2 "josh-connectors:PMOD_HOST" H 6300 2300 50  0001 C CNN
 F 3 "~" H 6300 2300 50  0001 C CNN
 	1    6300 2300
@@
 F 0 "J3" H 6375 4067 50  0000 C CNN
 F 1 "PMOD" H 6375 3976 50  0000 C CNN
-F 2 "josh-footprints:PMOD_HOST" H 6325 3650 50  0001 C CNN
+F 2 "josh-connectors:PMOD_HOST" H 6325 3650 50  0001 C CNN
 F 3 "~" H 6325 3650 50  0001 C CNN
 	1    6325 3650
@@
 NoConn ~ 4825 2375
 NoConn ~ 3775 2875
+$Comp
+L josh-mechnanical:Feather J1
+U 1 1 5D167D65
+P 4275 2775
+F 0 "J1" H 4300 3740 50  0000 C CNN
+F 1 "Feather" H 4300 3649 50  0000 C CNN
+F 2 "josh-connectors:featherwing" H 4475 1825 50  0001 C CNN
+F 3 "" H 4475 1825 50  0001 C CNN
+	1    4275 2775
+	1    0    0    -1
+$EndComp
 $EndSCHEMATC

Commit message: fixing things which broke resulting from library change
Parts:
- removed J1: Feather, josh-connectors:featherwing, symbol josh-mechnanical:Feather
- added J1: Feather, josh-connectors:featherwing, symbol josh-connector:Feather
Connections:
- net +3V3: now also J1.2 (3V3)
- net GND: now also J1.16 (NC), J1.4 (GND)
- net P1_1: now also J1.12 (IO7|MOSI)
- net P1_10: now also J1.5 (IO0)
- net P1_2: now also J1.10 (IO5)
- net P1_3: now also J1.8 (IO3)
- net P1_4: now also J1.6 (IO1)
- net P1_7: now also J1.11 (IO6|SCK)
- net P1_8: now also J1.9 (IO4)
- net P1_9: now also J1.7 (IO2)
- net P2_1: now also J1.17 (IO11|SDA)
- net P2_10: now also J1.24 (IO18)
- net P2_2: now also J1.19 (IO13)
- net P2_3: now also J1.21 (IO15)
- net P2_4: now also J1.23 (IO17)
- net P2_7: now also J1.18 (IO12|SCL)
- net P2_8: now also J1.20 (IO14)
- net P2_9: now also J1.22 (IO16)
Changed lines of the file:
@@
 NoConn ~ 3775 2875
 $Comp
-L josh-mechnanical:Feather J1
-U 1 1 5D167D65
+L josh-connector:Feather J1
+U 1 1 5D2CB6BF
 P 4275 2775
 F 0 "J1" H 4300 3740 50  0000 C CNN
