File: hardware/iCE40-fpga/iCE40-fpga.sch (KiCad schematic (older format))
At the start: 59 parts, among them J1 USB_B_Micro, J2 JST_PH, J3 Feather, Q1 DMP2045U, SW1 SW_Push, U1 MCP73831-2-OT, U2 TPD2S017, U3 AP2112K-3.3, U4 AT25SF081-SSHD-X, U5 AP2112K-1.2, U6 ICE40UP5K-SG48ITR, X1 DSC6101CI1A

Commit message: fixed footprints + added extra feather headers
Parts:
- removed C12: 100n, Capacitor_SMD:C_0603_1608Metric, symbol Device:C
- removed C13, C20, C25, C9: 1u, Capacitor_SMD:C_0603_1608Metric, symbol Device:C
- removed C14, C15, C23: 10n, Capacitor_SMD:C_0603_1608Metric, symbol Device:C
- removed U2: TPD2S017, Package_TO_SOT_SMD:SOT-23-6, symbol Power_Protection:TPD2S017
- added J4: Bonus_Row, josh-footprints:PinSocket_1x05_P2.54mm_Vertical_No_Markings, symbol Connector_Generic:Conn_01x05
- C8: value 1u -> 100n
- U6: footprint Package_DFN_QFN:QFN-48-1EP_7x7mm_P0.5mm_EP5.6x5.6mm -> josh-footprints:QFN-48-1EP_7x7mm_P0.5mm_EP5.3x5.3mm_ThermalVias
Connections:
- net labels added: USB_N, USB_P
- net labels removed: USB_DM, USB_DP
- wire segments 250 -> 208
Other:
- moved on the sheet: C10, C11, C16, C17, C18, C19, C21, C22, C24, D4, FB1, R11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

Commit message: all nets routed
Parts:
- removed C17: 10u, Capacitor_SMD:C_0603_1608Metric, symbol Device:C
- removed D3: GRN, LED_SMD:LED_0603_1608Metric, symbol Device:LED
- removed J4: Bonus_Row, josh-footprints:PinSocket_1x05_P2.54mm_Vertical_No_Markings, symbol Connector_Generic:Conn_01x05
- removed R10, R12, R9: 1K, Resistor_SMD:R_0603_1608Metric, symbol Device:R
- removed R11: 10K, Resistor_SMD:R_0603_1608Metric, symbol Device:R
- removed SW1: SW_Push, josh-footprints:Small_Tact_Switch, symbol Switch:SW_Push
- removed U4: AT25SF081-SSHD-X, Package_SO:SOIC-8_3.9x4.9mm_P1.27mm, symbol josh-symbols:AT25SF081-SSHD-X
- added RN3: 1K, Resistor_SMD:R_Array_Convex_4x0402, symbol Device:R_Pack04
- added U2: W25Q32JVZP, josh-footprints:WSON-8-1EP_6x5mm_P1.27mm_EP3.4x4.3mm, symbol josh-symbols:W25Q32JVZP
- D6: value LED_RGBA -> LTST-C19HE1WT; footprint josh-footprints:ARGB_PLCC4_1210_LED -> josh-footprints:0606LED
- R5: value 2K2 -> 10K
Connections:
- net labels added: IO0, IO1, IO10, IO11, IO12, IO13, IO14, IO15, IO16, IO17, IO18, IO19, IO2, IO3, IO4, IO5, IO6, IO7, IO8, IO9
- net labels removed: ICE_CRESET
- wire segments 208 -> 252
- no-connect marks 2 -> 5
Other:
- note removed: "iCE RESET Button"
- moved on the sheet: C7, D6

Commit message: cleaned up routing
Changed lines of the file:
@@
 Wire Wire Line
 	10050 1050 10275 1050
-Text Label 6625 3375 0    50   ~ 0
+Text Label 6625 3575 0    50   ~ 0
 nLED
 $Comp
@@
 Wire Wire Line
 	10900 5225 10625 5225
+Text Label 6425 2300 0    50   ~ 0
+IO4
+Wire Wire Line
+	6425 2300 6900 2300
 Text Label 6425 1700 0    50   ~ 0
-IO4
+IO5
 Wire Wire Line
 	6425 1700 6900 1700
-Text Label 6425 1800 0    50   ~ 0
-IO5
-Wire Wire Line
-	6425 1800 6900 1800
-Text Label 6425 2200 0    50   ~ 0
+Text Label 6425 2000 0    50   ~ 0
 IO6
 Wire Wire Line
-	6425 2200 6900 2200
+	6425 2000 6900 2000
 Text Label 10900 5125 2    50   ~ 0
 IO6
 Wire Wire Line
 	10900 5125 10625 5125
-Text Label 10900 5025 2    50   ~ 0
-IO7
-Wire Wire Line
-	10900 5025 10625 5025
-Text Label 6425 2000 0    50   ~ 0
-IO7
-Wire Wire Line
-	6425 2000 6900 2000
 Text Label 9300 5425 0    50   ~ 0
 IO19
@@
 Wire Wire Line
 	10900 4825 10625 4825
-Text Label 10900 4725 2    50   ~ 0
-IO10
-Wire Wire Line
-	10900 4725 10625 4725
 Text Label 8800 1850 2    50   ~ 0
 IO19
@@
 Wire Wire Line
 	6625 3775 6900 3775
-Text Label 6625 3575 0    50   ~ 0
+Text Label 6625 3375 0    50   ~ 0
 IO11
 Wire Wire Line
+	6625 3375 6900 3375
+Text Label 6425 1800 0    50   ~ 0
+IO8
+Text Label 6625 2200 0    50   ~ 0
+IO9
+Wire Wire Line
+	6625 2200 6900 2200
+Wire Wire Line
+	6425 1800 6900 1800
+Wire Wire Line
 	6625 3575 6900 3575
-Text Label 6425 2300 0    50   ~ 0
-IO8
-Text Label 6625 3675 0    50   ~ 0
-IO9
-Wire Wire Line
-	6625 3675 6900 3675
+Wire Wire Line
+	10900 4725 10625 4725
+Text Label 10900 4725 2    50   ~ 0
+IO10
+Wire Wire Line
+	10900 5025 10625 5025
+Text Label 10900 5025 2    50   ~ 0
+IO7
+Wire Wire Line
+	6625 3475 6900 3475
 Text Label 6625 3475 0    50   ~ 0
 IO10
 Wire Wire Line
-	6625 3475 6900 3475
-Wire Wire Line
-	6425 2300 6900 2300
-Wire Wire Line
-	6625 3375 6900 3375
+	6425 3675 6900 3675
+Text Label 6425 3675 0    50   ~ 0
+IO7
 $EndSCHEMATC

Commit message: added tx, rx leds, 7 segment and pmod wings
Parts:
- added D3, D8: GRN, LED_SMD:LED_0603_1608Metric, symbol Device:LED
- added RN4: 330R, Resistor_SMD:R_Array_Convex_4x0402, symbol Device:R_Pack04
- J3: symbol josh-symbols:Feather -> iCE40-fpga-rescue:Feather-josh-symbols
- RN3: value 1K -> 330R
Connections:
- wire segments 252 -> 262
- no-connect marks 5 -> 9
Other:
- note added: "UART LEDs"

Commit message: updated board + pmod
Connections:
- net labels removed: VBUS
- wire segments 262 -> 265
- no-connect marks 9 -> 16
Changed lines of the file:
@@
 Text Label 6625 3575 0    50   ~ 0
 nLED
-$Comp
-L power:VBUS #PWR06
-U 1 1 6009B446
-P 1150 1150
-F 0 "#PWR06" H 1150 1000 50  0001 C CNN
-F 1 "VBUS" H 1165 1323 50  0000 C CNN
-F 2 "" H 1150 1150 50  0001 C CNN
-F 3 "" H 1150 1150 50  0001 C CNN
-	1    1150 1150
-	1    0    0    -1
-$EndComp
 Text Label 9025 1200 2    50   ~ 0
 nICE_CRESET
@@
 Text Label 4300 2125 2    50   ~ 0
 RX_FPGA
-Text Label 9150 1950 2    50   ~ 0
+Text Label 9025 1950 2    50   ~ 0
 TX_FPGA
 Text Label 6425 1300 0    50   ~ 0
@@
 	1    0    0    -1
 $EndComp
-Wire Wire Line
-	975  3100 625  3100
 Connection ~ 625  3100
 Wire Wire Line
@@
 	9575 4500 9250 4500
 Wire Wire Line
-	1750 3425 2350 3425
+	1750 3425 2075 3425
 Connection ~ 1750 3425
 $Comp
@@
 $EndComp
 Wire Wire Line
-	1150 1150 1150 1200
-Wire Wire Line
 	1150 1200 1150 1475
-Connection ~ 1150 1200
 Wire Wire Line
 	1150 1200 1200 1200
@@
 NoConn ~ 10775 2000
 NoConn ~ 10775 2400
-Wire Wire Line
-	2575 5475 3700 5475
 $Comp
 L Device:R_Pack04 RN1
@@
 	2575 5275 3700 5275
 Wire Wire Line
-	3425 5375 2575 5375
-Wire Wire Line
-	3700 5375 3425 5375
-Connection ~ 3425 5375
-Wire Wire Line
-	3425 4925 3425 5375
-Wire Wire Line
 	2575 4975 3525 4975
 Wire Wire Line
@@
 Wire Wire Line
 	3225 5075 3700 5075
-NoConn ~ 3325 4925
 Wire Wire Line
 	6425 1300 6900 1300
 Wire Wire Line
-	9150 1950 8525 1950
+	9025 1950 8525 1950
 Text Label 10900 4600 2    50   ~ 0
 IO0
@@
 Wire Wire Line
 	10900 3700 10625 3700
-Text Label 8800 1850 2    50   ~ 0
+Text Label 9025 1850 2    50   ~ 0
 IO19
 Wire Wire Line
-	8800 1850 8525 1850
-Text Label 8800 1750 2    50   ~ 0
+	9025 1850 8525 1850
+Text Label 9025 1750 2    50   ~ 0
 IO18
 Wire Wire Line
-	8800 1750 8525 1750
-Text Label 8800 1650 2    50   ~ 0
+	9025 1750 8525 1750
+Text Label 9025 1650 2    50   ~ 0
 IO17
 Wire Wire Line
-	8800 1650 8525 1650
-Text Label 8800 1550 2    50   ~ 0
+	9025 1650 8525 1650
+Text Label 9025 1550 2    50   ~ 0
 IO16
 Wire Wire Line
-	8800 1550 8525 1550
-Text Label 8800 1450 2    50   ~ 0
+	9025 1550 8525 1550
+Text Label 9025 1450 2    50   ~ 0
 IO15
 Wire Wire Line
-	8800 1450 8525 1450
+	9025 1450 8525 1450
 Text Label 6625 3875 0    50   ~ 0
 IO14
@@
 Text Label 6425 1800 0    50   ~ 0
 IO8
-Text Label 6625 2200 0    50   ~ 0
+Text Label 6425 2200 0    50   ~ 0
 IO9
 Wire Wire Line
-	6625 2200 6900 2200
+	6425 2200 6900 2200
 Wire Wire Line
 	6425 1800 6900 1800
@@
 IO10
 Wire Wire Line
-	6425 3675 6900 3675
-Text Label 6425 3675 0    50   ~ 0
+	6625 3675 6900 3675
+Text Label 6625 3675 0    50   ~ 0
 IO7
 $Comp
@@
 NoConn ~ 10400 6150
 NoConn ~ 10400 5950
+NoConn ~ 6900 1900
+NoConn ~ 6900 2400
+NoConn ~ 6900 2500
+NoConn ~ 8525 2350
+NoConn ~ 8525 2250
+NoConn ~ 8525 2150
+NoConn ~ 8525 2050
+NoConn ~ 6900 3275
+Wire Wire Line
+	625  3100 975  3100
+$Comp
+L power:PWR_FLAG #FLG0101
+U 1 1 5D253666
+P 2075 3400
+F 0 "#FLG0101" H 2075 3475 50  0001 C CNN
+F 1 "PWR_FLAG" H 2075 3573 50  0000 C CNN
+F 2 "" H 2075 3400 50  0001 C CNN
+F 3 "~" H 2075 3400 50  0001 C CNN
+	1    2075 3400
+	1    0    0    -1
+$EndComp
+Wire Wire Line
+	2075 3400 2075 3425
+Connection ~ 2075 3425
+Wire Wire Line
+	2075 3425 2350 3425
+Wire Wire Line
+	2575 5475 3425 5475
+Wire Wire Line
+	2575 5375 3325 5375
+Wire Wire Line
+	3325 4925 3325 5375
+Connection ~ 3325 5375
+Wire Wire Line
+	3325 5375 3700 5375
+Wire Wire Line
+	3425 4925 3425 5475
+Connection ~ 3425 5475
+Wire Wire Line
+	3425 5475 3700 5475
 $EndSCHEMATC
